File: RD40_electronics/RD40_display_SMD_V1/RD40_display_SMD.kicad_sch (KiCad schematic)
At the start: 40 parts, among them J1 USB_B_Micro, J2 USB_B_Micro, Q1 J3Y, Q2 J3Y, U1 ATmega328-AU, U2 ISP, U3 CH340C, U4 ESP-12F, U5 CH340C, Y1 16MHz

Commit message: SMD circuit diagram further completed
Parts:
- removed C1, C2: 12pF, symbol Device:C
- removed C10, C13: 10µF, symbol RD40_display_SMD-rescue:CP-Device
- removed C11, C15, C16: 10µF, symbol Device:C_Polarized
- removed C12, C14, C17, C3, C4, C5, C6, C7, C8, C9: 100nF, symbol Device:C
- removed J1, J2: USB_B_Micro, symbol Connector:USB_B_Micro
- removed Q1, Q2: J3Y, symbol Simulation_SPICE:NPN
- removed R1, R10, R11, R2, R3, R7, R8, R9: 10k, symbol Device:R
- removed R4, R5: 1k, symbol Device:R
- removed R6: 470, symbol Device:R
- removed U1: ATmega328-AU, Package_QFP:TQFP-32_7x7mm_P0.8mm, symbol RD40_display_SMD-rescue:ATmega328-AU-MCU_Microchip_ATmega
- removed U2: ISP, symbol RD40_display_SMD-rescue:2x3pin_connector-my_symbols
- removed U3, U5: CH340C, Package_SO:SOIC-16_3.9x9.9mm_P1.27mm, symbol Interface_USB:CH340G
- removed U4: ESP-12F, RF_Module:ESP-12E, symbol RF_Module:ESP-12F
- removed Y1: 16MHz, symbol Device:Crystal_GND24
- added C1, C2: 22µF, 25V, Capacitor_SMD:C_0805_2012Metric, symbol RD40_display_SMD-rescue:CP-Device
- added C3, C4: 47µF, 10V, Capacitor_SMD:C_1206_3216Metric, symbol RD40_display_SMD-rescue:CP-Device
- added C5, C6, C7, C8: 100µF, 6,3V, Capacitor_SMD:C_1206_3216Metric, symbol RD40_display_SMD-rescue:CP-Device
- added D3, D4: B5819W, Diode_SMD:D_SOD-123, symbol Device:D_Schottky
- added L1: secondary coil, Crystal:Crystal_SMD_3225-4Pin_3.2x2.5mm, symbol my_symbols:Coil
- added U1: AP1117-50, Package_TO_SOT_SMD:SOT-223-3_TabPin2, symbol Regulator_Linear:AP1117-50
- added U2: AP1117-33, Package_TO_SOT_SMD:SOT-223-3_TabPin2, symbol Regulator_Linear:AP1117-50
- D1, D2: value D_Schottky -> B5819W; footprint (none) -> Diode_SMD:D_SOD-123; LCSC (none) -> C8598
Connections:
- net +3.3V: now also C5.1, C6.1, C7.1, C8.1, U2.2 (VO)
- net +5V: now also C3.1, C4.1, U1.2 (VO); no longer D1.1 (K), D2.1 (K)
- net GND: now also D2.2 (A), C1.2, C2.2, C3.2, C4.2, C5.2, C6.2, C7.2, C8.2, D4.2 (A), U1.1 (GND), U2.1 (GND)
- net at D1.2 (A): now also D2.1 (K), L1.2
- new net: D3.2 (A), D4.1 (K), L1.1
- new net U_unreg: C1.1, C2.1, D1.1 (K), D3.1 (K), U1.3 (VI), U2.3 (VI)
- no-connect marks 31 -> 0
Other:
- added sheet ATmega328P (ATmega328P.kicad_sch)
- added sheet ESP-12F (ESP-12F.kicad_sch)
- added sheet LED_electronics (LED_electronics.kicad_sch)
- note added: "ESP-12F microcontroller"
- note added: "LED electronics"
- note added: "RD40_SMD"
- note added: "Rotating LED Display"
- note added: "power supply"
- note removed: "C=2*(CL-Cstray) CL = 9pF (crystal data sheet) Cstray = 4 pF (estimate)"
- note removed: "ESP8266-12F microcontroller"
- company: (none) -> Ludwin Monz
- title: (none) -> RD40_SMD
