File: RD40_electronics/RD40_PS_V1/RD40_PS_V1.kicad_pcb (KiCad board)
At the start: 2 copper layers, 120 x 120 mm, 25 parts, among them J1 Barrel_Jack_Switch_Pin3Ring, M1 Motor_DC, Q1 BC337, Q2 BC337, SW1 SW_DPDT_x2, U1 Pin-Connector, U10 LM317_TO-220, U2 Pin-Connector, U3 Pin-Connector, U4 Pin-Connector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

Commit message: minor additions to PCBs
Other:
- net class Default removed
- net class breit removed
- net class mittel removed
