File: RD40_electronics/RD40_display_V1/RD40_display_V1.kicad_pcb (KiCad board)
At the start: 2 copper layers, 120 x 120 mm, 32 parts, among them SW1 SW_Push, U1 FT232, U2 TPIC6C595, U3 TPIC6C595, U4 TPIC6C595, U5 TPIC6C595, U6 TPIC6C595, U7 A3144, U8 LM1117-3.3, U9 ESP8266_01s

Commit message: minor additions to PCBs
Other:
- net class 1mm removed
- net class 2mm removed
- net class Default removed
